File: hardware/BLE-BMS.sch (EAGLE design)
At the start: 88 parts, among them Q1 BSS138, U1 BQ7694040

Commit message: Firmware, test pack layouts.
Firmware is mostly working! Layouts are pretty good.
Other:
- note added: "3.3V I2C conversion"
- note added: "Add pull down to alert of 500k-1M"
- note added: "May want 100 ohm into regsource"
- note added: "May want 200 ohm resistor to pack +"
- note added: "Swap resistor to 2512: CSR2512C0R001F"
- note added: "Thermistors have internally trimmed 10k pull up Do we need these pulldowns?"
- note added: "These resistors are pulling TS2 and TS3 below their actual ground (VC5X, VC10X)"
- note added: "This fet is not high enough V"
- note added: "bq7694002, 15 cell, 0x08 I2C, 3.3V, no CRC"

Commit message: v2 with Charge/Discharge MOSFET control and cell balancing
Many changes. Added large MOSFETs and pack interface circuitry. Added
small MOSFETs for individual cell balancing/charging. Corrected
Thermistor pull down error. All FPs pass 1:1 check.
Parts:
- added C35, C36, C37, C38: 0.1uF, SparkFun-Capacitors:0.1UF-100V-10%(0603)
- added D10, D11, D12, D13, D14, D15, D16, D17, D18, D19, D20, D21, D22, D8, D9: 5.6V, SparkFun-DiscreteSemi:DIODE-ZENER3.3V
- added D23: RED, SparkFun-LED:LED-RED1206
- added D4: BAS16, SparkFun-DiscreteSemi:DIODESOD
- added D5: MMSZ5246B-7-F, SparkFun-DiscreteSemi:DIODE-ZENERSOD-123
- added D6: SMCJ75AFS, SparkFun-DiscreteSemi:TVSSMC
- added D7: ES3J, SparkFun-DiscreteSemi:DIODESMC/DO-214AB
- added Q2, Q3: PSMN7R0-100BS, SparkFun-DiscreteSemi:MOSFET-NCHANNELPSMN7R0
- added Q4: 30V, 2.5A, SparkFun-DiscreteSemi:MOSFET-PCHANNELDMG2307L
- added R35, R7, R9: 1M, SparkFun-Resistors:1MOHM1/10W1%(0603)
- added R36, R67: 1K, SparkFun-Resistors:1KOHM1/10W1%(0603)
- added R37, R39, R40, R42, R44, R46, R48, R50, R52, R54, R56, R58, R60, R62, R64: 10K, SparkFun-Resistors:10KOHM1/10W1%(0603)0603
- added R38, R41, R43, R45, R47, R49, R51, R53, R55, R57, R59, R61, R63, R65: 100/.25W, SparkFun-Resistors:100OHM1/10W1%(0603)
- added R8: CSR2512C0R001F, bq769x0:RESISTOR2512
- added SJ5: JUMPER-PAD-2-NC_BY_TRACE, SparkFun-Passives:JUMPER-PAD-2-NC_BY_TRACE
- added U2, U3, U4, U5, U6, U7, U8, U9: DMP2240, SparkFun-DiscreteSemi:MOSFET-PCHANNEL_DUALSOT26
- R25: value 4.7k -> 1M; device SparkFun-Resistors:4.7KOHM1/10W1%(0603) -> SparkFun-Resistors:1MOHM1/10W1%(0603)
- R29: value .001 -> 100/.25W; device bq769x0:RESISTORWSR -> SparkFun-Resistors:100OHM1/10W1%(0603)
- U1: value BQ7694040 -> bq7694002DBT
Connections:
- removed net PACK-: R28.1, R29.2
- new net CHG_CTL: D4.C, D5.C, Q3.G, R25.2, R35.1
- new net LOAD-: C36.2, C37.1, D5.A, D7.A, Q3.S, R25.1
- new net LOAD1: Q2.D, Q3.D
- new net LOAD2: C35.1, Q2.S, R27.1, R8.1, R9.1
- new net N$1: D8.A, R37.1, U2G1.G
- new net N$12: D10.A, R40.1, U3G1.G
- new net N$13: R41.1, U3G1.D
- new net N$14: D11.A, R42.1, U3G2.G
- new net N$16: R43.1, U3G2.D
- new net N$18: D12.A, R44.1, U4G1.G
- new net N$19: R45.1, U4G1.D
- new net N$2: Q4.D, R36.2
- new net N$20: D13.A, R46.1, U4G2.G
- new net N$21: R47.1, U4G2.D
- new net N$23: R49.1, U5G1.D
- new net N$25: D14.A, R48.1, U5G1.G
- new net N$26: R51.1, U5G2.D
- new net N$27: D15.A, R50.1, U5G2.G
- new net N$37: R53.1, U6G1.D
- new net N$38: D16.A, R52.1, U6G1.G
- new net N$39: D17.A, R54.1, U6G2.G
- new net N$4: R29.1, U2G1.D
- new net N$41: R55.1, U6G2.D
- new net N$42: D18.A, R56.1, U7G1.G
- new net N$43: R57.1, U7G1.D
- new net N$44: D19.A, R58.1, U7G2.G
- new net N$46: R59.1, U7G2.D
- new net N$47: D20.A, R60.1, U8G1.G
- new net N$5: D9.A, R39.1, U2G2.G
- new net N$50: R61.1, U8G1.D
- new net N$51: D21.A, R62.1, U8G2.G
- new net N$52: R63.1, U8G2.D
- new net N$53: D22.A, R64.1, U9G1.G
- new net N$54: R65.1, U9G1.D
- new net N$57: D23.A, R67.1
- new net N$58: R67.2, SJ5.1
- new net N$6: C35.2, C36.1
- new net N$7: D4.A, R35.2, R36.1
- new net N$8: R38.1, U2G2.D
- new net N$9: C37.2, C38.1
- net ALERT: now also R7.2; no longer R25.2
- net CELL1: now also D8.C, R38.2, U2G1.S
- net CELL10: now also D17.C, R57.2, U6G2.S
- net CELL11: now also D18.C, R59.2, U7G1.S
- net CELL12: now also D19.C, R61.2, U7G2.S
- net CELL13: now also D20.C, R63.2, U8G1.S
- net CELL14: now also D21.C, R65.2, U8G2.S
- net CELL2: now also D9.C, R41.2, U2G2.S
- net CELL3: now also D10.C, R43.2, U3G1.S
- net CELL4: now also D11.C, R45.2, U3G2.S
- net CELL5: now also D12.C, R47.2, U4G1.S
- net CELL6: now also D13.C, R49.2, U4G2.S
- net CELL7: now also D14.C, R51.2, U5G1.S
- net CELL8: now also D15.C, R53.2, U5G2.S
- net CELL9: now also D16.C, R55.2, U6G1.S
- net CHG: now also Q4.S
- net DSG: now also Q2.G, R9.2
- net GND: now also D23.C, D6.A, Q4.G, R28.1, R29.2, R7.1, R8.2; no longer R25.1, R27.1, R29.1, R33.1, R34.1
- net PACK+: now also C38.2, D22.C, D6.C, D7.C, U9G1.S
- net REGOUT: now also SJ5.2
- net VC1: now also R37.2
- net VC10: now also R54.2
- net VC10X: now also R34.1
- net VC11: now also R56.2
- net VC12: now also R58.2
- net VC13: now also R60.2
- net VC14: now also R62.2
- net VC15: now also R64.2
- net VC2: now also R39.2
- net VC3: now also R40.2
- net VC4: now also R42.2
- net VC5: now also R44.2
- net VC5X: now also R33.1
- net VC6: now also R46.2
- net VC7: now also R48.2
- net VC8: now also R50.2
- net VC9: now also R52.2
Other:
- note added: "100 ohm 1/4 0603 : RHM100DCT-ND"
- note added: "100A NChan MOSFETs x 10 : 568-9705-1-ND"
- note added: "16V Zener x 10 : MMSZ5246B-FDICT-ND"
- note added: "3.3V is output only"
- note added: "Added CHG/DSG MOSFETs"
- note added: "Added charging FETs"
- note added: "Added footprint for 2512 resistor CSR2512C0R001F"
- note added: "Alert pull down changed to 1M"
- note added: "Changes on v1.1:"
- note added: "Charging FETs: DMP2240UDMDICT-ND"
- note added: "Check / narrow bq FP"
- note added: "Extra"
- note added: "Fixed pull downs on TS pins"
- note added: "Flyback diode: MURS360T3G / ES3JCT-ND"
- note added: "I2C Address: 0x08 I2C, no CRC"
- note added: "LOAD+"
- note added: "Max output is 50mA"
- note added: "N. Seidle"
- note added: "PACK-"
- note added: "Power"
- note added: "Smaller 2W resistor : CSR2512C0R001F"
- note added: "TVS Diode x 10: SMCJ75AFSCT-ND"
- note added: "To buy:"
- note added: "bq Main IC x 5 : 296-37788-5-ND"
- note removed: "Add pull down to alert of 500k-1M"
- note removed: "LOAD-"
- note removed: "Swap resistor to 2512: CSR2512C0R001F"
- note removed: "Thermistors have internally trimmed 10k pull up Do we need these pulldowns?"
- note removed: "These resistors are pulling TS2 and TS3 below their actual ground (VC5X, VC10X)"
- note removed: "bq7694002, 15 cell, 0x08 I2C, 3.3V, no CRC"
- moved on the sheet: C1, C10, C11, C12, C13, C14, C15, C16, C17, C18, C19, C2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
